Commit message: Optimised state machine and chessboard spawn logic

File: baxter/baxter/baxter_simulator/baxter_sim_examples/models/cafe_table/cafe_table.xacro (robot description, xacro)
@@ -33,5 +33,5 @@
   </link>
   <joint name="cafe_table_fixed" type="fixed">
-    <origin rpy="0 0 0" xyz="1.0 0 -0.93"/>
+    <origin rpy="0 0 0" xyz="0.78 0.3 -0.93"/>
     <axis xyz="0 0 1"/>
     <parent link="world"/>
